File: circuit/rocketry_circuit.kicad_sch (KiCad schematic)
At the start: 24 parts, among them J1 BATTERY, J2 E220-900T22D, J3 BMP280, J4 MPU6050, J5 Micro_SD_Card, J6 NEO-6M, U1 AMS1117-3.3, U2 SN74LVC125AD

Commit message: Footprint for resistors R1 R2
Parts:
- R1, R2: footprint Resistor_THT:R_Axial_DIN0204_L3.6mm_D1.6mm_P5.08mm_Horizontal -> Resistor_THT:R_Axial_DIN0207_L6.3mm_D2.5mm_P7.62mm_Horizontal
Changed lines of the file:
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@@
       (effects (font (size 1.27 1.27)))
     )
-    (property "Footprint" "Resistor_THT:R_Axial_DIN0204_L3.6mm_D1.6mm_P5.08mm_Horizontal" (at 124.46 33.528 90)
+    (property "Footprint" "Resistor_THT:R_Axial_DIN0207_L6.3mm_D2.5mm_P7.62mm_Horizontal" (at 124.46 33.528 90)
       (effects (font (size 1.27 1.27)) hide)
     )
@@
       (effects (font (size 1.27 1.27)))
     )
-    (property "Footprint" "Resistor_THT:R_Axial_DIN0204_L3.6mm_D1.6mm_P5.08mm_Horizontal" (at 134.62 43.688 90)
-      (effects (font (size 1.27 1.27)) hide)
-    )
+    (property "Footprint" "Resistor_THT:R_Axial_DIN0207_L6.3mm_D2.5mm_P7.62mm_Horizontal" (at 134.62 43.688 90)
+      (effects (font (size 1.27 1.27)) hide)
+    )
